Commit message: laser scan functionality added

File: xacro/barista_robot_model.urdf.xacro (robot description, xacro)
@@ -5,4 +5,5 @@
 <xacro:include filename="$(find barista_robot_description)/xacro/standoff_rod.xacro" />
 <xacro:include filename="$(find barista_robot_description)/xacro/cup_holder_tray.xacro" />
+<xacro:include filename="$(find barista_robot_description)/xacro/laser_scanner.xacro" />
   <material name="red">
       <color rgba="1.0 0.0 0.0 1"/>
@@ -132,3 +133,46 @@
     </plugin>
 </gazebo>
+<xacro:arg name="include_laser" default="true"/>
+<xacro:if value="$(arg include_laser)">
+  <xacro:laser_scanner laser_scanner_name="laser_scanner"/>
+  <joint name="laser_scanner_joint" type="fixed">
+    <origin rpy="0 0 0" xyz="0 0 0.1"/>
+    <parent link="chassis"/>
+    <child link="laser_scanner"/>
+  </joint>
+</xacro:if>
+ <!-- Enable Sensors in Gazebo Sim -->
+<gazebo>
+    <plugin filename="gz-sim-sensors-system" name="gz::sim::systems::Sensors">
+        <!-- use ogre2 if ogre v2.x is installed, otherwise use ogre -->
+        <render_engine>ogre2</render_engine>
+    </plugin>
+</gazebo>
+<!-- Laser Scanner Plugin -->
+<gazebo reference="laser_scanner">
+    <sensor type="gpu_lidar" name="gpu_lidar">
+        <pose relative_to='laser_scanner'>0 0 0 0 0 0</pose>
+        <gz_frame_id>laser_scanner</gz_frame_id>
+        <always_on>1</always_on>
+        <visualize>true</visualize>
+        <update_rate>100</update_rate>
+        <!-- change topic name from laser_scan to scan-->
+        <topic>scan</topic>
+        <ray>
+            <scan>
+                <horizontal>
+                    <samples>200</samples>
+                    <resolution>1</resolution>
+                    <min_angle>-3.14</min_angle>
+                    <max_angle>3.14</max_angle>
+                </horizontal>
+            </scan>
+            <range>
+                <min>0.1</min>
+                <max>5.0</max>
+                <resolution>0.01</resolution>
+            </range>
+        </ray>
+    </sensor>
+</gazebo>
 </robot>
