Commit message: fixed the topic name from laser_scan to scan. Currently will try to create one launch file that will set everything up.

File: urdf/barista_robot_model.urdf (robot description, URDF)
Before this commit: robot barista, 15 links, 14 joints
Links:
- added link laser_scan_frame, mass 0.05; collision cylinder length=0.04 radius=0.03; visual cylinder length=0.04 radius=0.03
Joints:
- added joint laser_scan_joint: type fixed, parent chassis, child laser_scan_frame, origin xyz=0 0 0.1 rpy=0 0 0

Commit message: task1 fixes

File: urdf/barista_robot_model.urdf (robot description, URDF)
Before this commit: robot barista, 16 links, 15 joints
Links:
- link laser_scan_frame: geometry collision mesh filename=file:///home/user/ros2_ws/src/cp7_auxiliary_files/meshes/in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; visual mesh filename=file:///home/user/ros2_ws/src/cp7_auxiliary_files/meshes/in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
Joints:
- joint laser_scan_joint: origin xyz=0 0 0.1 rpy=0 0 0 -> xyz=0.14 0.02 0.1 rpy=0 0 0
- joint left_cone_joint: origin xyz=0.07 0.135 0.1875 rpy=0 0 0 -> xyz=0.07 0.095 0.1875 rpy=0 0 0
- joint left_cone_joint2: origin xyz=-0.07 0.135 0.1875 rpy=0 0 0 -> xyz=-0.07 0.095 0.1875 rpy=0 0 0
- joint right_cone_joint: origin xyz=0.07 -0.135 0.1875 rpy=0 0 0 -> xyz=0.07 -0.095 0.1875 rpy=0 0 0
- joint right_cone_joint2: origin xyz=-0.07 -0.135 0.1875 rpy=0 0 0 -> xyz=-0.07 -0.095 0.1875 rpy=0 0 0

Commit message: made fixes on task2 and fixed positioning for scanner

File: urdf/barista_robot_model.urdf (robot description, URDF)
Before this commit: robot barista, 16 links, 15 joints
Joints:
- joint laser_scan_joint: origin xyz=0.14 0.02 0.1 rpy=0 0 0 -> xyz=0.14 0.02 0.087 rpy=0 0 0

File: xacro/barista_robot_model.urdf.xacro (robot description, xacro)
@@ -84,5 +84,5 @@
 <xacro:standoff_rod rod_name = "right2_rod"/>
 <joint name = "left_rod_joint" type = "fixed">
-    <origin rpy="0 0 0" xyz="0.07 0.135 0.1875"/>
+    <origin rpy="0 0 0" xyz="0.07 0.095 0.1875"/>
     <child link="left1_rod"/>
     <parent link="chassis"/>
@@ -90,5 +90,5 @@
 </joint>
 <joint name = "left_cone_joint2" type = "fixed">
-    <origin rpy="0 0 0" xyz="-0.07 0.135 0.1875"/>
+    <origin rpy="0 0 0" xyz="-0.07 0.095 0.1875"/>
     <child link="left2_rod"/>
     <parent link="chassis"/>
@@ -96,5 +96,5 @@
 </joint>
 <joint name = "right_cone_joint" type = "fixed">
-    <origin rpy="0 0 0" xyz="0.07 -0.135 0.1875"/>
+    <origin rpy="0 0 0" xyz="0.07 -0.095 0.1875"/>
     <child link="right1_rod"/>
     <parent link="chassis"/>
@@ -102,5 +102,5 @@
 </joint>
 <joint name = "right_cone_joint2" type = "fixed">
-    <origin rpy="0 0 0" xyz="-0.07 -0.135 0.1875"/>
+    <origin rpy="0 0 0" xyz="-0.07 -0.095 0.1875"/>
     <child link="right2_rod"/>
     <parent link="chassis"/>
@@ -137,17 +137,9 @@
   <xacro:laser_scanner laser_scanner_name="laser_scanner"/>
   <joint name="laser_scanner_joint" type="fixed">
-    <origin rpy="0 0 0" xyz="0 0 0.1"/>
+    <origin rpy="0 0 0" xyz="0.14 0.02 0.087"/>
     <parent link="chassis"/>
     <child link="laser_scanner"/>
   </joint>
-</xacro:if>
- <!-- Enable Sensors in Gazebo Sim -->
-<gazebo>
-    <plugin filename="gz-sim-sensors-system" name="gz::sim::systems::Sensors">
-        <!-- use ogre2 if ogre v2.x is installed, otherwise use ogre -->
-        <render_engine>ogre2</render_engine>
-    </plugin>
-</gazebo>
-<!-- Laser Scanner Plugin -->
+  <!-- Laser Scanner Plugin -->
 <gazebo reference="laser_scanner">
     <sensor type="gpu_lidar" name="gpu_lidar">
@@ -176,3 +168,11 @@
     </sensor>
 </gazebo>
+</xacro:if>
+ <!-- Enable Sensors in Gazebo Sim -->
+<gazebo>
+    <plugin filename="gz-sim-sensors-system" name="gz::sim::systems::Sensors">
+        <!-- use ogre2 if ogre v2.x is installed, otherwise use ogre -->
+        <render_engine>ogre2</render_engine>
+    </plugin>
+</gazebo>
 </robot>

File: xacro/laser_scanner.xacro (robot description, xacro)
@@ -5,5 +5,5 @@
   <visual>
     <geometry>
-      <cylinder length="0.04" radius="0.03"/>
+      <mesh filename="file:///home/user/ros2_ws/src/cp7_auxiliary_files/meshes/intel_realsense_d435.dae"/>
     </geometry>
     <material name="red"/>
@@ -11,5 +11,5 @@
   <collision>
     <geometry>
-      <cylinder length="0.04" radius="0.03"/>
+      <mesh filename="file:///home/user/ros2_ws/src/cp7_auxiliary_files/meshes/intel_realsense_d435.dae"/>
     </geometry>
   </collision>
